File: plates/pcb/bottom/corne-bottom-plate.kicad_pcb (KiCad board)
At the start: 2 copper layers, 133.8 x 91.4 mm, 7 parts

Commit message: refactor: change silkscreen
Parts:
- removed G*** (x2): LOGO, kbd:corne-horizontal
