File: plates/pcb/top/corne-top-plate.kicad_pcb (KiCad board)
At the start: 2 copper layers, 132.9 x 91.4 mm, 28 parts, among them SW2 KEY_SWITCH

Commit message: refactor: change silkscreen
Parts:
- removed G*** (x2): LOGO, kbd:corne-logo-horizontal-mask
Other:
- board text added: "cort"
